Commit message: added shoulders to urdf

File: src/sparke_description/src/sparke.urdf.xacro (robot description, xacro)
@@ -5,4 +5,10 @@
 	<xacro:property name="base_width" value="0.11"/>
   <xacro:property name="base_height" value="0.065"/>
+  <xacro:property name="shoulder_length" value="0.034"/>
+	<xacro:property name="shoulder_width" value="0.0635"/>
+  <xacro:property name="shoulder_height" value="0.013"/>
+  <xacro:property name="leg_length" value="0.01"/>
+	<xacro:property name="leg_width" value="0.01"/>
+  <xacro:property name="leg_height" value="0.01"/>
 	<!-- Robot Base -->
   <link name="base_link">
@@ -17,9 +23,54 @@
   </link>
 	<!-- Robot Footprint -->
-  <!-- <link name="base_footprint"/>
+  <link name="base_footprint"/>
   <joint name="base_joint" type="fixed">
     <parent link="base_link"/>
     <child link="base_footprint"/>
     <origin xyz="0.0 0.0 0.0" rpy="0 0 0"/>
-  </joint> -->
+  </joint>
+  <!-- Shoulders -->
+  <xacro:macro name="shoulder" params="prefix x_reflect y_reflect x_pos y_pos z_pos">
+    <link name="${prefix}_link">
+      <visual>
+        <origin xyz="0 0 0" rpy="0 0 0"/>
+        <geometry>
+            <box size="${shoulder_length} ${shoulder_width} ${shoulder_height}"/>
+        </geometry>
+        <material name="Gray">
+          <color rgba="0.5 0.5 0.5 1.0"/>
+        </material>
+      </visual>
+    </link>
+    <joint name="${prefix}_joint" type="fixed">
+      <parent link="base_link"/>
+      <child link="${prefix}_link"/>
+      <origin xyz="${(x_pos - (shoulder_length/25)) * x_reflect} ${(y_pos + (shoulder_width/2)) * y_reflect} ${z_pos - (shoulder_height/2)}" rpy="0 0 0"/>
+      <axis xyz="0 1 0"/>
+    </joint>
+  </xacro:macro>
+  <!-- Legs -->
+  <xacro:macro name="leg" params="prefix x_reflect y_reflect x_pos y_pos z_pos">
+    <link name="${prefix}_link">
+      <visual>
+        <origin xyz="0 0 0" rpy="0 0 0"/>
+        <geometry>
+            <box size="${leg_length} ${leg_width} ${leg_height}"/>
+        </geometry>
+        <material name="Gray">
+          <color rgba="0.5 0.5 0.5 1.0"/>
+        </material>
+      </visual>
+    </link>
+    <joint name="${prefix}_joint" type="fixed">
+      <parent link="base_link"/>
+      <child link="${prefix}_link"/>
+      <origin xyz="${(x_pos - (leg_length/25)) * x_reflect} ${(y_pos + (leg_width/2)) * y_reflect} ${z_pos - (leg_height/2)}" rpy="0 0 0"/>
+      <axis xyz="0 1 0"/>
+    </joint>
+  </xacro:macro>
+  <xacro:shoulder prefix="fl_shoulder" x_reflect="1" y_reflect="1" x_pos="0.101" y_pos="${base_width/2}" z_pos="${base_height/2}"/>
+  <xacro:shoulder prefix="fr_shoulder" x_reflect="1" y_reflect="-1" x_pos="0.101" y_pos="${base_width/2}" z_pos="${base_height/2}"/>
+  <xacro:shoulder prefix="br_shoulder" x_reflect="-1" y_reflect="-1" x_pos="0.101" y_pos="${base_width/2}" z_pos="${base_height/2}"/>
+  <xacro:shoulder prefix="bl_shoulder" x_reflect="-1" y_reflect="1" x_pos="0.101" y_pos="${base_width/2}" z_pos="${base_height/2}"/>
+  <!-- <xacro:leg prefix="fl_leg" x_reflect="1" y_reflect="1" x_pos="0.101" y_pos="${base_width/2}" z_pos="${base_height/2}"/> -->
 </robot>

Commit message: added new measurements to urdf

File: src/sparke_description/src/sparke.urdf.xacro (robot description, xacro)
@@ -8,7 +8,14 @@
 	<xacro:property name="shoulder_width" value="0.0635"/>
   <xacro:property name="shoulder_height" value="0.013"/>
-  <xacro:property name="leg_length" value="0.01"/>
-	<xacro:property name="leg_width" value="0.01"/>
-  <xacro:property name="leg_height" value="0.01"/>
+  <xacro:property name="leg_length" value="0.125"/>
+	<xacro:property name="leg_width" value="0.040"/>
+  <xacro:property name="leg_height" value="0.027"/>
+  <xacro:property name="wrist_joint_radius" value="0.125"/>
+	<xacro:property name="wrist_joint_width" value="0.040"/>
+  <xacro:property name="wrist_length" value="0.135"/>
+	<xacro:property name="wrist_width" value="0.0325"/>
+  <xacro:property name="wrist_height" value="0.015"/>
+  <xacro:property name="foot_radius" value="0.015"/>
+	<xacro:property name="foot_width" value="0.01"/>
 	<!-- Robot Base -->
   <link name="base_link">
@@ -31,5 +38,5 @@
   <!-- Shoulders -->
   <xacro:macro name="shoulder" params="prefix x_reflect y_reflect x_pos y_pos z_pos">
-    <link name="${prefix}_link">
+    <link name="${prefix}_shoulder_link">
       <visual>
         <origin xyz="0 0 0" rpy="0 0 0"/>
@@ -44,5 +51,5 @@
     <joint name="${prefix}_joint" type="fixed">
       <parent link="base_link"/>
-      <child link="${prefix}_link"/>
+      <child link="${prefix}_shoulder_link"/>
       <origin xyz="${(x_pos - (shoulder_length/25)) * x_reflect} ${(y_pos + (shoulder_width/2)) * y_reflect} ${z_pos - (shoulder_height/2)}" rpy="0 0 0"/>
       <axis xyz="0 1 0"/>
@@ -51,5 +58,5 @@
   <!-- Legs -->
   <xacro:macro name="leg" params="prefix x_reflect y_reflect x_pos y_pos z_pos">
-    <link name="${prefix}_link">
+    <link name="${prefix}_leg_link">
       <visual>
         <origin xyz="0 0 0" rpy="0 0 0"/>
@@ -62,15 +69,15 @@
       </visual>
     </link>
-    <joint name="${prefix}_joint" type="fixed">
-      <parent link="base_link"/>
-      <child link="${prefix}_link"/>
+    <joint name="${prefix}_leg_joint" type="fixed">
+      <parent link="${prefix}_shoulder_link"/>
+      <child link="${prefix}_leg_link"/>
       <origin xyz="${(x_pos - (leg_length/25)) * x_reflect} ${(y_pos + (leg_width/2)) * y_reflect} ${z_pos - (leg_height/2)}" rpy="0 0 0"/>
       <axis xyz="0 1 0"/>
     </joint>
   </xacro:macro>
-  <xacro:shoulder prefix="fl_shoulder" x_reflect="1" y_reflect="1" x_pos="0.101" y_pos="${base_width/2}" z_pos="${base_height/2}"/>
-  <xacro:shoulder prefix="fr_shoulder" x_reflect="1" y_reflect="-1" x_pos="0.101" y_pos="${base_width/2}" z_pos="${base_height/2}"/>
-  <xacro:shoulder prefix="br_shoulder" x_reflect="-1" y_reflect="-1" x_pos="0.101" y_pos="${base_width/2}" z_pos="${base_height/2}"/>
-  <xacro:shoulder prefix="bl_shoulder" x_reflect="-1" y_reflect="1" x_pos="0.101" y_pos="${base_width/2}" z_pos="${base_height/2}"/>
+  <xacro:shoulder prefix="fl" x_reflect="1" y_reflect="1" x_pos="0.101" y_pos="${base_width/2}" z_pos="${base_height/2}"/>
+  <xacro:shoulder prefix="fr" x_reflect="1" y_reflect="-1" x_pos="0.101" y_pos="${base_width/2}" z_pos="${base_height/2}"/>
+  <xacro:shoulder prefix="br" x_reflect="-1" y_reflect="-1" x_pos="0.101" y_pos="${base_width/2}" z_pos="${base_height/2}"/>
+  <xacro:shoulder prefix="bl" x_reflect="-1" y_reflect="1" x_pos="0.101" y_pos="${base_width/2}" z_pos="${base_height/2}"/>
   <!-- <xacro:leg prefix="fl_leg" x_reflect="1" y_reflect="1" x_pos="0.101" y_pos="${base_width/2}" z_pos="${base_height/2}"/> -->
 </robot>

Commit message: version 0.1 of urdf

File: src/sparke_description/src/sparke.urdf.xacro (robot description, xacro)
@@ -11,11 +11,11 @@
 	<xacro:property name="leg_width" value="0.040"/>
   <xacro:property name="leg_height" value="0.027"/>
-  <xacro:property name="wrist_joint_radius" value="0.125"/>
-	<xacro:property name="wrist_joint_width" value="0.040"/>
+  <xacro:property name="elbow_radius" value="0.0135"/>
+	<xacro:property name="elbow_width" value="0.040"/>
   <xacro:property name="wrist_length" value="0.135"/>
 	<xacro:property name="wrist_width" value="0.0325"/>
   <xacro:property name="wrist_height" value="0.015"/>
   <xacro:property name="foot_radius" value="0.015"/>
-	<xacro:property name="foot_width" value="0.01"/>
+	<xacro:property name="foot_width" value="0.0325"/>
 	<!-- Robot Base -->
   <link name="base_link">
@@ -24,6 +24,6 @@
         <box size="${base_length} ${base_width} ${base_height}"/>
       </geometry>
-      <material name="Cyan">
-        <color rgba="0.0 1.0 1.0 1.0"/>
+      <material name="Body">
+        <color rgba="0 0.5 0.5 1"/>
       </material>
     </visual>
@@ -44,6 +44,6 @@
             <box size="${shoulder_length} ${shoulder_width} ${shoulder_height}"/>
         </geometry>
-        <material name="Gray">
-          <color rgba="0.5 0.5 0.5 1.0"/>
+        <material name="Shoulder">
+          <color rgba="0 0.6 0.6 1.0"/>
         </material>
       </visual>
@@ -64,5 +64,5 @@
             <box size="${leg_length} ${leg_width} ${leg_height}"/>
         </geometry>
-        <material name="Gray">
+        <material name="Body">
           <color rgba="0.5 0.5 0.5 1.0"/>
         </material>
@@ -72,5 +72,59 @@
       <parent link="${prefix}_shoulder_link"/>
       <child link="${prefix}_leg_link"/>
-      <origin xyz="${(x_pos - (leg_length/25)) * x_reflect} ${(y_pos + (leg_width/2)) * y_reflect} ${z_pos - (leg_height/2)}" rpy="0 0 0"/>
+      <origin xyz="${(x_pos - (leg_length/25)) * x_reflect} ${(y_pos + (leg_width/2)) * y_reflect} ${z_pos - (leg_height/2)}" rpy="0 ${-pi/4} 0"/>
+      <axis xyz="0 1 0"/>
+    </joint>
+    <link name="${prefix}_elbow_link">
+      <visual>
+        <origin xyz="0 0 0" rpy="0 ${pi/2} 0"/>
+        <geometry>
+            <cylinder radius="${elbow_radius}" length="${elbow_width}"/>
+        </geometry>
+        <material name="Body">
+          <color rgba="0.5 0.5 0.5 1.0"/>
+        </material>
+      </visual>
+    </link>
+    <joint name="${prefix}_elbow_joint" type="fixed">
+      <parent link="${prefix}_leg_link"/>
+      <child link="${prefix}_elbow_link"/>
+      <origin xyz="${-leg_length/2} 0 0" rpy="0 0 ${pi/2}"/>
+      <axis xyz="0 1 0"/>
+    </joint>
+  </xacro:macro>
+  <!-- Wrists -->
+  <xacro:macro name="wrist" params="prefix x_reflect y_reflect x_pos y_pos z_pos">
+    <link name="${prefix}_wrist_link">
+      <visual>
+        <origin xyz="0 0 0" rpy="0 0 0"/>
+        <geometry>
+            <box size="${wrist_length} ${wrist_width} ${wrist_height}"/>
+        </geometry>
+        <material name="Gray">
+          <color rgba="0.5 0.5 0.5 1.0"/>
+        </material>
+      </visual>
+    </link>
+    <joint name="${prefix}_wrist_joint" type="fixed">
+      <parent link="${prefix}_elbow_link"/>
+      <child link="${prefix}_wrist_link"/>
+      <origin xyz="0 0 ${-wrist_length/2}" rpy="0 ${pi/2} ${pi/2}"/>
+      <axis xyz="0 1 0"/>
+    </joint>
+    <link name="${prefix}_foot_link">
+      <visual>
+        <origin xyz="0 0 0" rpy="0 0 0"/>
+        <geometry>
+            <cylinder radius="${foot_radius}" length="${foot_width+0.001}"/>
+        </geometry>
+        <material>
+          <color rgba="0.1 0.1 0.1 1"/>
+        </material>
+      </visual>
+    </link>
+    <joint name="${prefix}_foot_joint" type="fixed">
+      <parent link="${prefix}_wrist_link"/>
+      <child link="${prefix}_foot_link"/>
+      <origin xyz="${wrist_length/2} 0 0" rpy="0 ${pi/2} ${pi/2}"/>
       <axis xyz="0 1 0"/>
     </joint>
@@ -80,4 +134,11 @@
   <xacro:shoulder prefix="br" x_reflect="-1" y_reflect="-1" x_pos="0.101" y_pos="${base_width/2}" z_pos="${base_height/2}"/>
   <xacro:shoulder prefix="bl" x_reflect="-1" y_reflect="1" x_pos="0.101" y_pos="${base_width/2}" z_pos="${base_height/2}"/>
-  <!-- <xacro:leg prefix="fl_leg" x_reflect="1" y_reflect="1" x_pos="0.101" y_pos="${base_width/2}" z_pos="${base_height/2}"/> -->
+  <xacro:leg prefix="fl" x_reflect="1" y_reflect="1" x_pos="${-(leg_length/2)+(shoulder_length*0.9)}" y_pos="${-leg_width/2}" z_pos="${-(leg_length/4)-(shoulder_height/4)}"/>
+  <xacro:leg prefix="fr" x_reflect="1" y_reflect="1" x_pos="${-(leg_length/2)+(shoulder_length*0.9)}" y_pos="${-leg_width/2}" z_pos="${-(leg_length/4)-(shoulder_height/4)}"/>
+  <xacro:leg prefix="br" x_reflect="1" y_reflect="1" x_pos="${-(leg_length/2)+(shoulder_length*0.9)}" y_pos="${-leg_width/2}" z_pos="${-(leg_length/4)-(shoulder_height/4)}"/>
+  <xacro:leg prefix="bl" x_reflect="1" y_reflect="1" x_pos="${-(leg_length/2)+(shoulder_length*0.9)}" y_pos="${-leg_width/2}" z_pos="${-(leg_length/4)-(shoulder_height/4)}"/>
+  <xacro:wrist prefix="fl" x_reflect="1" y_reflect="1" x_pos="0" y_pos="0" z_pos="0"/>
+  <xacro:wrist prefix="fr" x_reflect="1" y_reflect="1" x_pos="0" y_pos="0" z_pos="0"/>
+  <xacro:wrist prefix="br" x_reflect="1" y_reflect="1" x_pos="0" y_pos="0" z_pos="0"/>
+  <xacro:wrist prefix="bl" x_reflect="1" y_reflect="1" x_pos="0" y_pos="0" z_pos="0"/>
 </robot>

Commit message: added gazebo compatibility and basic teleop simulation controls

File: src/sparke_description/src/sparke.urdf.xacro (robot description, xacro)
@@ -18,4 +18,25 @@
   <xacro:property name="foot_radius" value="0.015"/>
 	<xacro:property name="foot_width" value="0.0325"/>
+  <!-- Define intertial property macros  -->
+  <xacro:macro name="box_inertia" params="m w h d">
+    <inertial>
+      <origin xyz="0 0 0" rpy="${pi/2} 0 ${pi/2}"/>
+      <mass value="${m}"/>
+      <inertia ixx="${(m/12) * (h*h + d*d)}" ixy="0.0" ixz="0.0" iyy="${(m/12) * (w*w + d*d)}" iyz="0.0" izz="${(m/12) * (w*w + h*h)}"/>
+    </inertial>
+  </xacro:macro>
+  <xacro:macro name="cylinder_inertia" params="m r h">
+    <inertial>
+      <origin xyz="0 0 0" rpy="${pi/2} 0 0" />
+      <mass value="${m}"/>
+      <inertia ixx="${(m/12) * (3*r*r + h*h)}" ixy = "0" ixz = "0" iyy="${(m/12) * (3*r*r + h*h)}" iyz = "0" izz="${(m/2) * (r*r)}"/>
+    </inertial>
+  </xacro:macro>
+  <xacro:macro name="sphere_inertia" params="m r">
+    <inertial>
+      <mass value="${m}"/>
+      <inertia ixx="${(2/5) * m * (r*r)}" ixy="0.0" ixz="0.0" iyy="${(2/5) * m * (r*r)}" iyz="0.0" izz="${(2/5) * m * (r*r)}"/>
+    </inertial>
+  </xacro:macro>
 	<!-- Robot Base -->
   <link name="base_link">
@@ -28,5 +49,20 @@
       </material>
     </visual>
+    <collision>
+      <geometry>
+        <box size="${base_length} ${base_width} ${base_height}"/>
+      </geometry>
+    </collision>
+    <xacro:box_inertia m="15" w="${base_width}" d="${base_length}" h="${base_height}"/>
   </link>
+  <gazebo>
+    <plugin name="object_controller" filename="libgazebo_ros_planar_move.so">
+      <commandTopic>cmd_vel</commandTopic>
+      <odometryTopic>odom</odometryTopic>
+      <odometryFrame>odom</odometryFrame>
+      <odometryRate>20.0</odometryRate>
+      <robotBaseFrame>base_footprint</robotBaseFrame>
+    </plugin>
+  </gazebo>
 	<!-- Robot Footprint -->
   <link name="base_footprint"/>
@@ -48,4 +84,10 @@
         </material>
       </visual>
+      <collision>
+        <geometry>
+          <box size="${shoulder_length} ${shoulder_width} ${shoulder_height}"/>
+        </geometry>
+      </collision>
+      <xacro:box_inertia m="0.1" w="${shoulder_length}" d="${shoulder_width}" h="${shoulder_height}"/>
     </link>
     <joint name="${prefix}_joint" type="fixed">
@@ -68,4 +110,10 @@
         </material>
       </visual>
+      <collision>
+        <geometry>
+          <box size="${leg_length} ${leg_width} ${leg_height}"/>
+        </geometry>
+      </collision>
+      <xacro:box_inertia m="0.5" w="${leg_length}" d="${leg_width}" h="${leg_height}"/>
     </link>
     <joint name="${prefix}_leg_joint" type="fixed">
@@ -85,4 +133,10 @@
         </material>
       </visual>
+      <collision>
+        <geometry>
+          <cylinder radius="${elbow_radius}" length="${elbow_width}"/>
+        </geometry>
+      </collision>
+      <xacro:cylinder_inertia m="0.1" r="${elbow_radius}" h="${elbow_width}"/>
     </link>
     <joint name="${prefix}_elbow_joint" type="fixed">
@@ -105,4 +159,10 @@
         </material>
       </visual>
+      <collision>
+        <geometry>
+          <box size="${wrist_length} ${wrist_width} ${wrist_height}"/>
+        </geometry>
+      </collision>
+      <xacro:box_inertia m="0.4" w="${wrist_length}" d="${wrist_width}" h="${wrist_height}"/>
     </link>
     <joint name="${prefix}_wrist_joint" type="fixed">
@@ -118,8 +178,14 @@
             <cylinder radius="${foot_radius}" length="${foot_width+0.001}"/>
         </geometry>
-        <material>
+        <material name="black">
           <color rgba="0.1 0.1 0.1 1"/>
         </material>
       </visual>
+      <collision>
+        <geometry>
+          <cylinder radius="${foot_radius}" length="${foot_width}"/>
+        </geometry>
+      </collision>
+      <xacro:cylinder_inertia m="0.1" r="${foot_radius}" h="${foot_width}"/>
     </link>
     <joint name="${prefix}_foot_joint" type="fixed">
@@ -129,4 +195,8 @@
       <axis xyz="0 1 0"/>
     </joint>
+    <gazebo reference="${prefix}_foot_link">
+      <mu1>0.0</mu1>
+      <mu2>0.0</mu2>
+    </gazebo>
   </xacro:macro>
   <xacro:shoulder prefix="fl" x_reflect="1" y_reflect="1" x_pos="0.101" y_pos="${base_width/2}" z_pos="${base_height/2}"/>

Commit message: added lidar to urdf

File: src/sparke_description/src/sparke.urdf.xacro (robot description, xacro)
@@ -72,4 +72,62 @@
     <origin xyz="0.0 0.0 0.0" rpy="0 0 0"/>
   </joint>
+  <link name="lidar_link">
+    <inertial>
+      <origin xyz="0 0 0" rpy="0 0 0"/>
+      <mass value="0.125"/>
+      <inertia ixx="0.001"  ixy="0"  ixz="0" iyy="0.001" iyz="0" izz="0.001" />
+    </inertial>
+    <collision>
+      <origin xyz="0 0 0" rpy="0 0 0"/>
+      <geometry>
+        <cylinder radius="0.0508" length="0.055"/>
+      </geometry>
+    </collision>
+    <visual>
+      <origin xyz="0 0 0" rpy="0 0 0"/>
+      <geometry>
+        <cylinder radius="0.0508" length="0.055"/>
+      </geometry>
+    </visual>
+  </link>
+  <joint name="lidar_joint" type="fixed">
+    <parent link="base_link"/>
+    <child link="lidar_link"/>
+    <origin xyz="0 0 ${(base_height/2)+(0.055/2)}" rpy="0 0 0"/>
+  </joint>
+  <gazebo reference="lidar_link">
+    <sensor name="lidar" type="ray">
+      <always_on>true</always_on>
+      <visualize>true</visualize>
+      <update_rate>5</update_rate>
+      <ray>
+        <scan>
+          <horizontal>
+            <samples>360</samples>
+            <resolution>1.000000</resolution>
+            <min_angle>0.000000</min_angle>
+            <max_angle>6.280000</max_angle>
+          </horizontal>
+        </scan>
+        <range>
+          <min>0.120000</min>
+          <max>3.5</max>
+          <resolution>0.015000</resolution>
+        </range>
+        <noise>
+          <type>gaussian</type>
+          <mean>0.0</mean>
+          <stddev>0.01</stddev>
+        </noise>
+      </ray>
+      <plugin name="scan" filename="libgazebo_ros_ray_sensor.so">
+        <ros>
+          <remapping>~/out:=scan</remapping>
+        </ros>
+        <output_type>sensor_msgs/LaserScan</output_type>
+        <frame_name>lidar_link</frame_name>
+      </plugin>
+    </sensor>
+  </gazebo>
   <!-- Shoulders -->
   <xacro:macro name="shoulder" params="prefix x_reflect y_reflect x_pos y_pos z_pos">

Commit message: fixed base_footprint to base_link transform

File: src/sparke_description/src/sparke.urdf.xacro (robot description, xacro)
@@ -68,6 +68,6 @@
   <link name="base_footprint"/>
   <joint name="base_joint" type="fixed">
-    <parent link="base_link"/>
-    <child link="base_footprint"/>
+    <parent link="base_footprint"/>
+    <child link="base_link"/>
     <origin xyz="0.0 0.0 0.0" rpy="0 0 0"/>
   </joint>
