Commit message: added cameras to urdf, adjustment still needed

File: src/sparke_description/src/sparke.urdf.xacro (robot description, xacro)
@@ -130,4 +130,159 @@
     </sensor>
   </gazebo>
+  <!-- Stereo Camera -->
+  <link name="stereo_camera_link">
+    <visual>
+      <origin xyz="0 0 0" rpy="0 0 0"/>
+      <geometry>
+        <box size="0.01 0.06 0.02"/>
+      </geometry>
+      <material name="camera_base">
+        <color rgba="1 1 1 1"/>
+      </material>
+    </visual>
+    <collision>
+      <geometry>
+        <box size="0.01 0.06 0.02"/>
+      </geometry>
+    </collision>
+    <xacro:box_inertia m="0.01" w="0" d="0" h="0"/>
+  </link>
+  <joint name="stereo_camera_joint" type="fixed">
+    <parent link="base_link"/>
+    <child link="stereo_camera_link"/>
+    <origin xyz="${base_length/2} 0 0" rpy="0 0 0"/>
+    <axis xyz="0 1 0"/>
+  </joint>
+  <!-- Camera -->
+  <link name="r_camera_link">
+    <collision>
+      <origin xyz="0 0 0" rpy="0 0 0"/>
+      <geometry>
+        <cylinder radius="0.005" length="0.01"/>
+      </geometry>
+    </collision>
+    <visual>
+      <origin xyz="0 0 0" rpy="0 0 0"/>
+      <geometry>
+        <cylinder radius="0.005" length="0.01"/>
+      </geometry>
+      <material name="red"/>
+    </visual>
+    <inertial>
+      <mass value="1e-5" />
+      <origin xyz="0 0 0" rpy="0 0 0"/>
+      <inertia ixx="1e-6" ixy="0" ixz="0" iyy="1e-6" iyz="0" izz="1e-6" />
+    </inertial>
+  </link>
+  <joint name="r_camera_joint" type="fixed">
+    <axis xyz="0 1 0" />
+    <origin xyz="0.01 -0.02 0" rpy="0 ${pi/2} 0"/>
+    <parent link="stereo_camera_link"/>
+    <child link="r_camera_link"/>
+  </joint>
+  <link name="l_camera_link">
+    <collision>
+      <origin xyz="0 0 0" rpy="0 0 0"/>
+      <geometry>
+        <cylinder radius="0.005" length="0.01"/>
+      </geometry>
+    </collision>
+    <visual>
+      <origin xyz="0 0 0" rpy="0 0 0"/>
+      <geometry>
+        <cylinder radius="0.005" length="0.01"/>
+      </geometry>
+      <material name="red"/>
+    </visual>
+    <inertial>
+      <mass value="1e-5" />
+      <origin xyz="0 0 0" rpy="0 0 0"/>
+      <inertia ixx="1e-6" ixy="0" ixz="0" iyy="1e-6" iyz="0" izz="1e-6" />
+    </inertial>
+  </link>
+  <joint name="l_camera_joint" type="fixed">
+    <axis xyz="0 1 0" />
+    <origin xyz="0.01 0.02 0" rpy="0 ${pi/2} 0"/>
+    <parent link="stereo_camera_link"/>
+    <child link="l_camera_link"/>
+  </joint>
+  <gazebo reference="r_camera_link">
+    <sensor type="camera" name="camera1">
+      <update_rate>30.0</update_rate>
+      <camera name="r_camera">
+        <horizontal_fov>1.3962634</horizontal_fov>
+        <image>
+          <width>800</width>
+          <height>800</height>
+          <format>R8G8B8</format>
+        </image>
+        <clip>
+          <near>0.02</near>
+          <far>300</far>
+        </clip>
+        <noise>
+          <type>gaussian</type>
+          <!-- Noise is sampled independently per pixel on each frame.
+               That pixel's noise value is added to each of its color
+               channels, which at that point lie in the range [0,1]. -->
+          <mean>0.0</mean>
+          <stddev>0.007</stddev>
+        </noise>
+      </camera>
+      <plugin name="camera_controller" filename="libgazebo_ros_camera.so">
+        <alwaysOn>true</alwaysOn>
+        <updateRate>0.0</updateRate>
+        <cameraName>sparke/camera1</cameraName>
+        <imageTopicName>image_raw</imageTopicName>
+        <cameraInfoTopicName>camera_info</cameraInfoTopicName>
+        <frameName>camera_link</frameName>
+        <hackBaseline>0.07</hackBaseline>
+        <distortionK1>0.0</distortionK1>
+        <distortionK2>0.0</distortionK2>
+        <distortionK3>0.0</distortionK3>
+        <distortionT1>0.0</distortionT1>
+        <distortionT2>0.0</distortionT2>
+      </plugin>
+    </sensor>
+  </gazebo>
+  <gazebo reference="l_camera_link">
+    <sensor type="camera" name="camera2">
+      <update_rate>30.0</update_rate>
+      <camera name="l_camera">
+        <horizontal_fov>1.3962634</horizontal_fov>
+        <image>
+          <width>800</width>
+          <height>800</height>
+          <format>R8G8B8</format>
+        </image>
+        <clip>
+          <near>0.02</near>
+          <far>300</far>
+        </clip>
+        <noise>
+          <type>gaussian</type>
+          <!-- Noise is sampled independently per pixel on each frame.
+               That pixel's noise value is added to each of its color
+               channels, which at that point lie in the range [0,1]. -->
+          <mean>0.0</mean>
+          <stddev>0.007</stddev>
+        </noise>
+      </camera>
+      <plugin name="camera_controller" filename="libgazebo_ros_camera.so">
+        <alwaysOn>true</alwaysOn>
+        <updateRate>0.0</updateRate>
+        <cameraName>sparke/camera2</cameraName>
+        <imageTopicName>image_raw</imageTopicName>
+        <cameraInfoTopicName>camera_info</cameraInfoTopicName>
+        <frameName>camera_link</frameName>
+        <hackBaseline>0.07</hackBaseline>
+        <distortionK1>0.0</distortionK1>
+        <distortionK2>0.0</distortionK2>
+        <distortionK3>0.0</distortionK3>
+        <distortionT1>0.0</distortionT1>
+        <distortionT2>0.0</distortionT2>
+      </plugin>
+    </sensor>
+  </gazebo>
   <!-- Shoulders -->
   <xacro:macro name="shoulder" params="prefix x_reflect y_reflect x_pos y_pos z_pos">

Commit message: joint control started

File: src/sparke_description/src/sparke.urdf.xacro (robot description, xacro)
@@ -353,9 +353,11 @@
       <xacro:cylinder_inertia m="0.1" r="${elbow_radius}" h="${elbow_width}"/>
     </link>
-    <joint name="${prefix}_elbow_joint" type="fixed">
+    <joint name="${prefix}_elbow_joint" type="revolute">
       <parent link="${prefix}_leg_link"/>
       <child link="${prefix}_elbow_link"/>
       <origin xyz="${-leg_length/2} 0 0" rpy="0 0 ${pi/2}"/>
-      <axis xyz="0 1 0"/>
+      <axis xyz="1 0 0"/>
+      <limit effort="1000.0" lower="-15" upper="15" velocity="30"/>
+      <dynamics damping="0.0" friction="0.0"/>
     </joint>
   </xacro:macro>
@@ -425,3 +427,22 @@
   <xacro:wrist prefix="br" x_reflect="1" y_reflect="1" x_pos="0" y_pos="0" z_pos="0"/>
   <xacro:wrist prefix="bl" x_reflect="1" y_reflect="1" x_pos="0" y_pos="0" z_pos="0"/>
+  <ros2_control name="GazeboSystem" type="system">
+    <hardware>
+      <plugin>gazebo_ros2_control/GazeboSystem</plugin>
+    </hardware>
+    <joint name="fl_elbow_joint">
+      <command_interface name="effort">
+        <param name="min">-1000</param>
+        <param name="max">1000</param>
+      </command_interface>
+      <state_interface name="position"/>
+      <state_interface name="velocity"/>
+      <state_interface name="effort"/>
+    </joint>
+  </ros2_control>
+  <gazebo>
+    <plugin filename="libgazebo_ros2_control.so" name="gazebo_ros2_control">
+      <parameters>$(find sparke_description)/params/sparke_controller_effort.yaml</parameters>
+    </plugin>
+  </gazebo>
 </robot>

Commit message: added 4 legs

File: src/sparke_description/src/sparke.urdf.xacro (robot description, xacro)
@@ -99,5 +99,5 @@
     <sensor name="lidar" type="ray">
       <always_on>true</always_on>
-      <visualize>true</visualize>
+      <visualize>false</visualize>
       <update_rate>5</update_rate>
       <ray>
@@ -358,5 +358,5 @@
       <origin xyz="${-leg_length/2} 0 0" rpy="0 0 ${pi/2}"/>
       <axis xyz="1 0 0"/>
-      <limit effort="1000.0" lower="-15" upper="15" velocity="30"/>
+      <limit effort="9.52" lower="${-pi/2}" upper="${pi/2}" velocity="9.52"/>
       <dynamics damping="0.0" friction="0.0"/>
     </joint>
@@ -410,8 +410,4 @@
       <axis xyz="0 1 0"/>
     </joint>
-    <gazebo reference="${prefix}_foot_link">
-      <mu1>0.0</mu1>
-      <mu2>0.0</mu2>
-    </gazebo>
   </xacro:macro>
   <xacro:shoulder prefix="fl" x_reflect="1" y_reflect="1" x_pos="0.101" y_pos="${base_width/2}" z_pos="${base_height/2}"/>
@@ -433,6 +429,33 @@
     <joint name="fl_elbow_joint">
       <command_interface name="effort">
-        <param name="min">-1000</param>
-        <param name="max">1000</param>
+        <param name="min">-100</param>
+        <param name="max">100</param>
+      </command_interface>
+      <state_interface name="position"/>
+      <state_interface name="velocity"/>
+      <state_interface name="effort"/>
+    </joint>
+    <joint name="bl_elbow_joint">
+      <command_interface name="effort">
+        <param name="min">-100</param>
+        <param name="max">100</param>
+      </command_interface>
+      <state_interface name="position"/>
+      <state_interface name="velocity"/>
+      <state_interface name="effort"/>
+    </joint>
+    <joint name="fr_elbow_joint">
+      <command_interface name="effort">
+        <param name="min">-100</param>
+        <param name="max">100</param>
+      </command_interface>
+      <state_interface name="position"/>
+      <state_interface name="velocity"/>
+      <state_interface name="effort"/>
+    </joint>
+    <joint name="br_elbow_joint">
+      <command_interface name="effort">
+        <param name="min">-100</param>
+        <param name="max">100</param>
       </command_interface>
       <state_interface name="position"/>
