Commit message: trying to stop robot from glitching around

File: src/sparke_description/src/sparke.urdf.xacro (robot description, xacro)
@@ -54,17 +54,10 @@
       </geometry>
     </collision>
-    <xacro:box_inertia m="15" w="${base_width}" d="${base_length}" h="${base_height}"/>
+    <xacro:box_inertia m="1" w="${base_width}" d="${base_length}" h="${base_height}"/>
   </link>
-  <gazebo>
-    <plugin name="object_controller" filename="libgazebo_ros_planar_move.so">
-      <commandTopic>cmd_vel</commandTopic>
-      <odometryTopic>odom</odometryTopic>
-      <odometryFrame>odom</odometryFrame>
-      <odometryRate>20.0</odometryRate>
-      <robotBaseFrame>base_footprint</robotBaseFrame>
-    </plugin>
-  </gazebo>
 	<!-- Robot Footprint -->
-  <link name="base_footprint"/>
+  <link name="base_footprint">
+    <xacro:box_inertia m="1" w="${base_width}" d="${base_length}" h="${base_height}"/>
+  </link>
   <joint name="base_joint" type="fixed">
     <parent link="base_footprint"/>
@@ -74,5 +67,4 @@
   <link name="lidar_link">
     <inertial>
-      <origin xyz="0 0 0" rpy="0 0 0"/>
       <mass value="0.125"/>
       <inertia ixx="0.001"  ixy="0"  ixz="0" iyy="0.001" iyz="0" izz="0.001" />
@@ -146,5 +138,5 @@
       </geometry>
     </collision>
-    <xacro:box_inertia m="0.01" w="0" d="0" h="0"/>
+    <xacro:box_inertia m="0.01" w="0.06" d="0.01" h="0.02"/>
   </link>
   <joint name="stereo_camera_joint" type="fixed">
@@ -171,5 +163,4 @@
     <inertial>
       <mass value="1e-5" />
-      <origin xyz="0 0 0" rpy="0 0 0"/>
       <inertia ixx="1e-6" ixy="0" ixz="0" iyy="1e-6" iyz="0" izz="1e-6" />
     </inertial>
@@ -197,5 +188,4 @@
     <inertial>
       <mass value="1e-5" />
-      <origin xyz="0 0 0" rpy="0 0 0"/>
       <inertia ixx="1e-6" ixy="0" ixz="0" iyy="1e-6" iyz="0" izz="1e-6" />
     </inertial>
@@ -230,5 +220,5 @@
         </noise>
       </camera>
-      <plugin name="camera_controller" filename="libgazebo_ros_camera.so">
+      <plugin name="r_camera_controller" filename="libgazebo_ros_camera.so">
         <alwaysOn>true</alwaysOn>
         <updateRate>0.0</updateRate>
@@ -269,5 +259,5 @@
         </noise>
       </camera>
-      <plugin name="camera_controller" filename="libgazebo_ros_camera.so">
+      <plugin name="l_camera_controller" filename="libgazebo_ros_camera.so">
         <alwaysOn>true</alwaysOn>
         <updateRate>0.0</updateRate>
@@ -287,9 +277,9 @@
   <!-- Shoulders -->
   <xacro:macro name="shoulder" params="prefix x_reflect y_reflect x_pos y_pos z_pos">
-    <link name="${prefix}_shoulder_link">
+    <link name="${prefix}_b2s_link">
       <visual>
         <origin xyz="0 0 0" rpy="0 0 0"/>
         <geometry>
-            <box size="${shoulder_length} ${shoulder_width} ${shoulder_height}"/>
+          <sphere radius="0.001"/>
         </geometry>
         <material name="Shoulder">
@@ -299,14 +289,41 @@
       <collision>
         <geometry>
+          <sphere radius="0.001"/>
+        </geometry>
+      </collision>
+      <xacro:sphere_inertia m="0.01" r="0.001"/>
+    </link>
+    <joint name="${prefix}_b2s_joint" type="revolute">
+      <parent link="base_link"/>
+      <child link="${prefix}_b2s_link"/>
+      <origin xyz="${(x_pos - (shoulder_length/25)) * x_reflect} ${(y_pos + (shoulder_width/2)) * y_reflect} ${z_pos - (shoulder_height/2)}" rpy="0 0 0"/>
+      <axis xyz="1 0 0"/>
+      <limit effort="1000" lower="0" upper="${pi/4}" velocity="9.52"/>
+      <dynamics damping="0.0" friction="1.0"/>
+    </joint>
+    <link name="${prefix}_shoulder_link">
+      <visual>
+        <origin xyz="0 0 0" rpy="0 0 0"/>
+        <geometry>
+            <box size="${shoulder_length} ${shoulder_width} ${shoulder_height}"/>
+        </geometry>
+        <material name="Shoulder">
+          <color rgba="0 0.6 0.6 1.0"/>
+        </material>
+      </visual>
+      <collision>
+        <geometry>
           <box size="${shoulder_length} ${shoulder_width} ${shoulder_height}"/>
         </geometry>
       </collision>
-      <xacro:box_inertia m="0.1" w="${shoulder_length}" d="${shoulder_width}" h="${shoulder_height}"/>
+      <xacro:box_inertia m="1" w="${shoulder_width}" d="${shoulder_length}" h="${shoulder_height}"/>
     </link>
-    <joint name="${prefix}_joint" type="fixed">
-      <parent link="base_link"/>
+    <joint name="${prefix}_shoulder_joint" type="revolute">
+      <parent link="${prefix}_b2s_link"/>
       <child link="${prefix}_shoulder_link"/>
-      <origin xyz="${(x_pos - (shoulder_length/25)) * x_reflect} ${(y_pos + (shoulder_width/2)) * y_reflect} ${z_pos - (shoulder_height/2)}" rpy="0 0 0"/>
+      <origin xyz="0 0 0" rpy="0 0 0"/>
       <axis xyz="0 1 0"/>
+      <limit effort="1000" lower="${-pi/2}" upper="${pi/2}" velocity="9.52"/>
+      <dynamics damping="0.0" friction="1.0"/>
     </joint>
   </xacro:macro>
@@ -325,8 +342,8 @@
       <collision>
         <geometry>
-          <box size="${leg_length} ${leg_width} ${leg_height}"/>
+          <box size="0 0 0"/>
         </geometry>
       </collision>
-      <xacro:box_inertia m="0.5" w="${leg_length}" d="${leg_width}" h="${leg_height}"/>
+      <xacro:box_inertia m="1" w="${leg_width}" d="${leg_length}" h="${leg_height}"/>
     </link>
     <joint name="${prefix}_leg_joint" type="fixed">
@@ -351,5 +368,5 @@
         </geometry>
       </collision>
-      <xacro:cylinder_inertia m="0.1" r="${elbow_radius}" h="${elbow_width}"/>
+      <xacro:cylinder_inertia m="1" r="${elbow_radius}" h="${elbow_width}"/>
     </link>
     <joint name="${prefix}_elbow_joint" type="revolute">
@@ -358,6 +375,6 @@
       <origin xyz="${-leg_length/2} 0 0" rpy="0 0 ${pi/2}"/>
       <axis xyz="1 0 0"/>
-      <limit effort="9.52" lower="${-pi/2}" upper="${pi/2}" velocity="9.52"/>
-      <dynamics damping="0.0" friction="0.0"/>
+      <limit effort="1000" lower="${-pi/2}" upper="${pi/2}" velocity="9.52"/>
+      <dynamics damping="0.0" friction="1.0"/>
     </joint>
   </xacro:macro>
@@ -376,8 +393,8 @@
       <collision>
         <geometry>
-          <box size="${wrist_length} ${wrist_width} ${wrist_height}"/>
+          <box size="0 0 0"/>
         </geometry>
       </collision>
-      <xacro:box_inertia m="0.4" w="${wrist_length}" d="${wrist_width}" h="${wrist_height}"/>
+      <xacro:box_inertia m="1" w="${wrist_width}" d="${wrist_length}" h="${wrist_height}"/>
     </link>
     <joint name="${prefix}_wrist_joint" type="fixed">
@@ -402,6 +419,12 @@
         </geometry>
       </collision>
-      <xacro:cylinder_inertia m="0.1" r="${foot_radius}" h="${foot_width}"/>
+      <xacro:cylinder_inertia m="1" r="${foot_radius}" h="${foot_width}"/>
     </link>
+    <gazebo reference="${prefix}_foot_link">
+      <mu>100</mu>
+      <mu2>50</mu2>
+      <kp  value="1000000.0" />
+      <kd  value="1.0" />
+    </gazebo>
     <joint name="${prefix}_foot_joint" type="fixed">
       <parent link="${prefix}_wrist_link"/>
@@ -428,36 +451,132 @@
     </hardware>
     <joint name="fl_elbow_joint">
-      <command_interface name="effort">
-        <param name="min">-100</param>
-        <param name="max">100</param>
-      </command_interface>
-      <state_interface name="position"/>
+      <command_interface name="position">
+        <param name="min">-1.57</param>
+        <param name="max">1.57</param>
+      </command_interface>
+      <state_interface name="position">
+        <param name="initial_value">0.0</param>
+      </state_interface>
+      <state_interface name="velocity"/>
+      <state_interface name="effort"/>
+    </joint>
+    <joint name="fr_elbow_joint">
+      <command_interface name="position">
+        <param name="min">-1.57</param>
+        <param name="max">1.57</param>
+      </command_interface>
+      <state_interface name="position">
+        <param name="initial_value">0.0</param>
+      </state_interface>
       <state_interface name="velocity"/>
       <state_interface name="effort"/>
     </joint>
     <joint name="bl_elbow_joint">
-      <command_interface name="effort">
-        <param name="min">-100</param>
-        <param name="max">100</param>
-      </command_interface>
-      <state_interface name="position"/>
-      <state_interface name="velocity"/>
-      <state_interface name="effort"/>
-    </joint>
-    <joint name="fr_elbow_joint">
-      <command_interface name="effort">
-        <param name="min">-100</param>
-        <param name="max">100</param>
-      </command_interface>
-      <state_interface name="position"/>
+      <command_interface name="position">
+        <param name="min">-1.57</param>
+        <param name="max">1.57</param>
+      </command_interface>
+      <state_interface name="position">
+        <param name="initial_value">0.0</param>
+      </state_interface>
       <state_interface name="velocity"/>
       <state_interface name="effort"/>
     </joint>
     <joint name="br_elbow_joint">
-      <command_interface name="effort">
-        <param name="min">-100</param>
-        <param name="max">100</param>
-      </command_interface>
-      <state_interface name="position"/>
+      <command_interface name="position">
+        <param name="min">-1.57</param>
+        <param name="max">1.57</param>
+      </command_interface>
+      <state_interface name="position">
+        <param name="initial_value">0.0</param>
+      </state_interface>
+      <state_interface name="velocity"/>
+      <state_interface name="effort"/>
+    </joint>
+    <joint name="fl_b2s_joint">
+      <command_interface name="position">
+        <param name="min">-1.57</param>
+        <param name="max">1.57</param>
+      </command_interface>
+      <state_interface name="position">
+        <param name="initial_value">0.0</param>
+      </state_interface>
+      <state_interface name="velocity"/>
+      <state_interface name="effort"/>
+    </joint>
+    <joint name="fr_b2s_joint">
+      <command_interface name="position">
+        <param name="min">-1.57</param>
+        <param name="max">1.57</param>
+      </command_interface>
+      <state_interface name="position">
+        <param name="initial_value">0.0</param>
+      </state_interface>
+      <state_interface name="velocity"/>
+      <state_interface name="effort"/>
+    </joint>
+    <joint name="bl_b2s_joint">
+      <command_interface name="position">
+        <param name="min">-1.57</param>
+        <param name="max">1.57</param>
+      </command_interface>
+      <state_interface name="position">
+        <param name="initial_value">0.0</param>
+      </state_interface>
+      <state_interface name="velocity"/>
+      <state_interface name="effort"/>
+    </joint>
+    <joint name="br_b2s_joint">
+      <command_interface name="position">
+        <param name="min">-1.57</param>
+        <param name="max">1.57</param>
+      </command_interface>
+      <state_interface name="position">
+        <param name="initial_value">0.0</param>
+      </state_interface>
+      <state_interface name="velocity"/>
+      <state_interface name="effort"/>
+    </joint>
+    <joint name="fl_shoulder_joint">
+      <command_interface name="position">
+        <param name="min">-1.57</param>
+        <param name="max">1.57</param>
+      </command_interface>
+      <state_interface name="position">
+        <param name="initial_value">0.0</param>
+      </state_interface>
+      <state_interface name="velocity"/>
+      <state_interface name="effort"/>
+    </joint>
+    <joint name="fr_shoulder_joint">
+      <command_interface name="position">
+        <param name="min">-1.57</param>
+        <param name="max">1.57</param>
+      </command_interface>
+      <state_interface name="position">
+        <param name="initial_value">0.0</param>
+      </state_interface>
+      <state_interface name="velocity"/>
+      <state_interface name="effort"/>
+    </joint>
+    <joint name="bl_shoulder_joint">
+      <command_interface name="position">
+        <param name="min">-1.57</param>
+        <param name="max">1.57</param>
+      </command_interface>
+      <state_interface name="position">
+        <param name="initial_value">0.0</param>
+      </state_interface>
+      <state_interface name="velocity"/>
+      <state_interface name="effort"/>
+    </joint>
+    <joint name="br_shoulder_joint">
+      <command_interface name="position">
+        <param name="min">-1.57</param>
+        <param name="max">1.57</param>
+      </command_interface>
+      <state_interface name="position">
+        <param name="initial_value">0.0</param>
+      </state_interface>
       <state_interface name="velocity"/>
       <state_interface name="effort"/>
@@ -465,7 +584,128 @@
   </ros2_control>
   <gazebo>
-    <plugin filename="libgazebo_ros2_control.so" name="gazebo_ros2_control">
-      <parameters>$(find sparke_description)/params/sparke_controller_effort.yaml</parameters>
+    <plugin name="gazebo_ros2_control" filename="libgazebo_ros2_control.so">
+      <robot_sim_type>gazebo_ros2_control/GazeboSystem</robot_sim_type>
+      <parameters>$(find sparke_description)/params/simple_controller.yaml</parameters>
     </plugin>
   </gazebo>
+  <transmission name="tran1">
+    <type>transmission_interface/SimpleTransmission</type>
+    <joint name="fl_elbow_joint">
+      <hardwareInterface>hardware_interface/PositionJointInterface</hardwareInterface>
+    </joint>
+    <actuator name="motor1">
+      <hardwareInterface>hardware_interface/PositionJointInterface</hardwareInterface>
+      <mechanicalReduction>1</mechanicalReduction>
+    </actuator>
+  </transmission>
+  <transmission name="tran2">
+    <type>transmission_interface/SimpleTransmission</type>
+    <joint name="fr_elbow_joint">
+      <hardwareInterface>hardware_interface/PositionJointInterface</hardwareInterface>
+    </joint>
+    <actuator name="motor2">
+      <hardwareInterface>hardware_interface/PositionJointInterface</hardwareInterface>
+      <mechanicalReduction>1</mechanicalReduction>
+    </actuator>
+  </transmission>
+  <transmission name="tran3">
+    <type>transmission_interface/SimpleTransmission</type>
+    <joint name="bl_elbow_joint">
+      <hardwareInterface>hardware_interface/PositionJointInterface</hardwareInterface>
+    </joint>
+    <actuator name="motor3">
+      <hardwareInterface>hardware_interface/PositionJointInterface</hardwareInterface>
+      <mechanicalReduction>1</mechanicalReduction>
+    </actuator>
+  </transmission>
+  <transmission name="tran4">
+    <type>transmission_interface/SimpleTransmission</type>
+    <joint name="br_elbow_joint">
+      <hardwareInterface>hardware_interface/PositionJointInterface</hardwareInterface>
+    </joint>
+    <actuator name="motor4">
+      <hardwareInterface>hardware_interface/PositionJointInterface</hardwareInterface>
+      <mechanicalReduction>1</mechanicalReduction>
+    </actuator>
+  </transmission>
+  <transmission name="tran5">
+    <type>transmission_interface/SimpleTransmission</type>
+    <joint name="fl_b2s_joint">
+      <hardwareInterface>hardware_interface/PositionJointInterface</hardwareInterface>
+    </joint>
+    <actuator name="motor5">
+      <hardwareInterface>hardware_interface/PositionJointInterface</hardwareInterface>
+      <mechanicalReduction>1</mechanicalReduction>
+    </actuator>
+  </transmission>
+  <transmission name="tran6">
+    <type>transmission_interface/SimpleTransmission</type>
+    <joint name="fr_b2s_joint">
+      <hardwareInterface>hardware_interface/PositionJointInterface</hardwareInterface>
+    </joint>
+    <actuator name="motor6">
+      <hardwareInterface>hardware_interface/PositionJointInterface</hardwareInterface>
+      <mechanicalReduction>1</mechanicalReduction>
+    </actuator>
+  </transmission>
+  <transmission name="tran7">
+    <type>transmission_interface/SimpleTransmission</type>
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