Commit message: possible fixes

File: src/sparke_description/src/sparke.urdf.xacro (robot description, xacro)
@@ -54,10 +54,24 @@
       </geometry>
     </collision>
-    <xacro:box_inertia m="1" w="${base_width}" d="${base_length}" h="${base_height}"/>
+    <xacro:box_inertia m="1.0" w="${base_width}" d="${base_length}" h="${base_height}"/>
   </link>
+  <gazebo reference="base_link">
+      <mu>50</mu>
+      <mu2>25</mu2>
+      <kp value="50000.0"/>
+      <kd value="0.05"/>
+      <dampingFactor value="0.0"/>
+    </gazebo>
 	<!-- Robot Footprint -->
   <link name="base_footprint">
-    <xacro:box_inertia m="1" w="${base_width}" d="${base_length}" h="${base_height}"/>
+    <xacro:box_inertia m="1.0" w="${base_width}" d="${base_length}" h="${base_height}"/>
   </link>
+  <gazebo reference="base_footprint">
+      <mu>50</mu>
+      <mu2>25</mu2>
+      <kp value="50000.0"/>
+      <kd value="0.05"/>
+      <dampingFactor value="0.0"/>
+  </gazebo>
   <joint name="base_joint" type="fixed">
     <parent link="base_footprint"/>
@@ -65,214 +79,4 @@
     <origin xyz="0.0 0.0 0.0" rpy="0 0 0"/>
   </joint>
-  <link name="lidar_link">
-    <inertial>
-      <mass value="0.125"/>
-      <inertia ixx="0.001"  ixy="0"  ixz="0" iyy="0.001" iyz="0" izz="0.001" />
-    </inertial>
-    <collision>
-      <origin xyz="0 0 0" rpy="0 0 0"/>
-      <geometry>
-        <cylinder radius="0.0508" length="0.055"/>
-      </geometry>
-    </collision>
-    <visual>
-      <origin xyz="0 0 0" rpy="0 0 0"/>
-      <geometry>
-        <cylinder radius="0.0508" length="0.055"/>
-      </geometry>
-    </visual>
-  </link>
-  <joint name="lidar_joint" type="fixed">
-    <parent link="base_link"/>
-    <child link="lidar_link"/>
-    <origin xyz="0 0 ${(base_height/2)+(0.055/2)}" rpy="0 0 0"/>
-  </joint>
-  <gazebo reference="lidar_link">
-    <sensor name="lidar" type="ray">
-      <always_on>true</always_on>
-      <visualize>false</visualize>
-      <update_rate>5</update_rate>
-      <ray>
-        <scan>
-          <horizontal>
-            <samples>360</samples>
-            <resolution>1.000000</resolution>
-            <min_angle>0.000000</min_angle>
-            <max_angle>6.280000</max_angle>
-          </horizontal>
-        </scan>
-        <range>
-          <min>0.120000</min>
-          <max>3.5</max>
-          <resolution>0.015000</resolution>
-        </range>
-        <noise>
-          <type>gaussian</type>
-          <mean>0.0</mean>
-          <stddev>0.01</stddev>
-        </noise>
-      </ray>
-      <plugin name="scan" filename="libgazebo_ros_ray_sensor.so">
-        <ros>
-          <remapping>~/out:=scan</remapping>
-        </ros>
-        <output_type>sensor_msgs/LaserScan</output_type>
-        <frame_name>lidar_link</frame_name>
-      </plugin>
-    </sensor>
-  </gazebo>
-  <!-- Stereo Camera -->
-  <link name="stereo_camera_link">
-    <visual>
-      <origin xyz="0 0 0" rpy="0 0 0"/>
-      <geometry>
-        <box size="0.01 0.06 0.02"/>
-      </geometry>
-      <material name="camera_base">
-        <color rgba="1 1 1 1"/>
-      </material>
-    </visual>
-    <collision>
-      <geometry>
-        <box size="0.01 0.06 0.02"/>
-      </geometry>
-    </collision>
-    <xacro:box_inertia m="0.01" w="0.06" d="0.01" h="0.02"/>
-  </link>
-  <joint name="stereo_camera_joint" type="fixed">
-    <parent link="base_link"/>
-    <child link="stereo_camera_link"/>
-    <origin xyz="${base_length/2} 0 0" rpy="0 0 0"/>
-    <axis xyz="0 1 0"/>
-  </joint>
-  <!-- Camera -->
-  <link name="r_camera_link">
-    <collision>
-      <origin xyz="0 0 0" rpy="0 0 0"/>
-      <geometry>
-        <cylinder radius="0.005" length="0.01"/>
-      </geometry>
-    </collision>
-    <visual>
-      <origin xyz="0 0 0" rpy="0 0 0"/>
-      <geometry>
-        <cylinder radius="0.005" length="0.01"/>
-      </geometry>
-      <material name="red"/>
-    </visual>
-    <inertial>
-      <mass value="1e-5" />
-      <inertia ixx="1e-6" ixy="0" ixz="0" iyy="1e-6" iyz="0" izz="1e-6" />
-    </inertial>
-  </link>
-  <joint name="r_camera_joint" type="fixed">
-    <axis xyz="0 1 0" />
-    <origin xyz="0.01 -0.02 0" rpy="0 ${pi/2} 0"/>
-    <parent link="stereo_camera_link"/>
-    <child link="r_camera_link"/>
-  </joint>
-  <link name="l_camera_link">
-    <collision>
-      <origin xyz="0 0 0" rpy="0 0 0"/>
-      <geometry>
-        <cylinder radius="0.005" length="0.01"/>
-      </geometry>
-    </collision>
-    <visual>
-      <origin xyz="0 0 0" rpy="0 0 0"/>
-      <geometry>
-        <cylinder radius="0.005" length="0.01"/>
-      </geometry>
-      <material name="red"/>
-    </visual>
-    <inertial>
-      <mass value="1e-5" />
-      <inertia ixx="1e-6" ixy="0" ixz="0" iyy="1e-6" iyz="0" izz="1e-6" />
-    </inertial>
-  </link>
-  <joint name="l_camera_joint" type="fixed">
-    <axis xyz="0 1 0" />
-    <origin xyz="0.01 0.02 0" rpy="0 ${pi/2} 0"/>
-    <parent link="stereo_camera_link"/>
-    <child link="l_camera_link"/>
-  </joint>
-  <gazebo reference="r_camera_link">
-    <sensor type="camera" name="camera1">
-      <update_rate>30.0</update_rate>
-      <camera name="r_camera">
-        <horizontal_fov>1.3962634</horizontal_fov>
-        <image>
-          <width>800</width>
-          <height>800</height>
-          <format>R8G8B8</format>
-        </image>
-        <clip>
-          <near>0.02</near>
-          <far>300</far>
-        </clip>
-        <noise>
-          <type>gaussian</type>
-          <!-- Noise is sampled independently per pixel on each frame.
-               That pixel's noise value is added to each of its color
-               channels, which at that point lie in the range [0,1]. -->
-          <mean>0.0</mean>
-          <stddev>0.007</stddev>
-        </noise>
-      </camera>
-      <plugin name="r_camera_controller" filename="libgazebo_ros_camera.so">
-        <alwaysOn>true</alwaysOn>
-        <updateRate>0.0</updateRate>
-        <cameraName>sparke/camera1</cameraName>
-        <imageTopicName>image_raw</imageTopicName>
-        <cameraInfoTopicName>camera_info</cameraInfoTopicName>
-        <frameName>camera_link</frameName>
-        <hackBaseline>0.07</hackBaseline>
-        <distortionK1>0.0</distortionK1>
-        <distortionK2>0.0</distortionK2>
-        <distortionK3>0.0</distortionK3>
-        <distortionT1>0.0</distortionT1>
-        <distortionT2>0.0</distortionT2>
-      </plugin>
-    </sensor>
-  </gazebo>
-  <gazebo reference="l_camera_link">
-    <sensor type="camera" name="camera2">
-      <update_rate>30.0</update_rate>
-      <camera name="l_camera">
-        <horizontal_fov>1.3962634</horizontal_fov>
-        <image>
-          <width>800</width>
-          <height>800</height>
-          <format>R8G8B8</format>
-        </image>
-        <clip>
-          <near>0.02</near>
-          <far>300</far>
-        </clip>
-        <noise>
-          <type>gaussian</type>
-          <!-- Noise is sampled independently per pixel on each frame.
-               That pixel's noise value is added to each of its color
-               channels, which at that point lie in the range [0,1]. -->
-          <mean>0.0</mean>
-          <stddev>0.007</stddev>
-        </noise>
-      </camera>
-      <plugin name="l_camera_controller" filename="libgazebo_ros_camera.so">
-        <alwaysOn>true</alwaysOn>
-        <updateRate>0.0</updateRate>
-        <cameraName>sparke/camera2</cameraName>
-        <imageTopicName>image_raw</imageTopicName>
-        <cameraInfoTopicName>camera_info</cameraInfoTopicName>
-        <frameName>camera_link</frameName>
-        <hackBaseline>0.07</hackBaseline>
-        <distortionK1>0.0</distortionK1>
-        <distortionK2>0.0</distortionK2>
-        <distortionK3>0.0</distortionK3>
-        <distortionT1>0.0</distortionT1>
-        <distortionT2>0.0</distortionT2>
-      </plugin>
-    </sensor>
-  </gazebo>
   <!-- Shoulders -->
   <xacro:macro name="shoulder" params="prefix x_reflect y_reflect x_pos y_pos z_pos">
@@ -281,5 +85,5 @@
         <origin xyz="0 0 0" rpy="0 0 0"/>
         <geometry>
-          <sphere radius="0.001"/>
+            <box size="${shoulder_length} ${shoulder_width} ${shoulder_height}"/>
         </geometry>
         <material name="Shoulder">
@@ -289,8 +93,8 @@
       <collision>
         <geometry>
-          <sphere radius="0.001"/>
+          <box size="${shoulder_length} ${shoulder_width} ${shoulder_height}"/>
         </geometry>
       </collision>
-      <xacro:sphere_inertia m="0.01" r="0.001"/>
+      <xacro:box_inertia m="1.0" w="${shoulder_width}" d="${shoulder_length}" h="${shoulder_height}"/>
     </link>
     <joint name="${prefix}_b2s_joint" type="revolute">
@@ -299,7 +103,14 @@
       <origin xyz="${(x_pos - (shoulder_length/25)) * x_reflect} ${(y_pos + (shoulder_width/2)) * y_reflect} ${z_pos - (shoulder_height/2)}" rpy="0 0 0"/>
       <axis xyz="1 0 0"/>
-      <limit effort="1000" lower="0" upper="${pi/4}" velocity="9.52"/>
-      <dynamics damping="0.0" friction="1.0"/>
-    </joint>
+      <limit effort="1000" lower="0" upper="${pi/4}" velocity="0.0"/>
+      <dynamics damping="0" friction="1"/>
+    </joint>
+    <gazebo reference="${prefix}_b2s_link">
+      <mu>50</mu>
+      <mu2>25</mu2>
+      <kp value="50000.0"/>
+      <kd value="0.05"/>
+      <dampingFactor value="0.0"/>
+    </gazebo>
     <link name="${prefix}_shoulder_link">
       <visual>
@@ -317,5 +128,5 @@
         </geometry>
       </collision>
-      <xacro:box_inertia m="1" w="${shoulder_width}" d="${shoulder_length}" h="${shoulder_height}"/>
+      <xacro:box_inertia m="1.0" w="${shoulder_width}" d="${shoulder_length}" h="${shoulder_height}"/>
     </link>
     <joint name="${prefix}_shoulder_joint" type="revolute">
@@ -324,7 +135,14 @@
       <origin xyz="0 0 0" rpy="0 0 0"/>
       <axis xyz="0 1 0"/>
-      <limit effort="1000" lower="${-pi/2}" upper="${pi/2}" velocity="9.52"/>
-      <dynamics damping="0.0" friction="1.0"/>
-    </joint>
+      <limit effort="1000" lower="${-pi/2}" upper="${pi/2}" velocity="0.0"/>
+      <dynamics damping="0" friction="1"/>
+    </joint>
+    <gazebo reference="${prefix}_shoulder_link">
+      <mu>50</mu>
+      <mu2>25</mu2>
+      <kp value="50000.0"/>
+      <kd value="0.05"/>
+      <dampingFactor value="0.0"/>
+    </gazebo>
   </xacro:macro>
   <!-- Legs -->
@@ -342,9 +160,16 @@
       <collision>
         <geometry>
-          <box size="0 0 0"/>
+          <box size="${leg_length} ${leg_width} ${leg_height}"/>
         </geometry>
       </collision>
-      <xacro:box_inertia m="1" w="${leg_width}" d="${leg_length}" h="${leg_height}"/>
+      <xacro:box_inertia m="1.0" w="${leg_width}" d="${leg_length}" h="${leg_height}"/>
     </link>
+    <gazebo reference="${prefix}_leg_link">
+      <mu>50</mu>
+      <mu2>25</mu2>
+      <kp value="50000.0"/>
+      <kd value="0.05"/>
+      <dampingFactor value="0.0"/>
+    </gazebo>
     <joint name="${prefix}_leg_joint" type="fixed">
       <parent link="${prefix}_shoulder_link"/>
@@ -365,9 +190,17 @@
       <collision>
         <geometry>
+          <origin xyz="0 0 0" rpy="0 ${pi/2} 0"/>
           <cylinder radius="${elbow_radius}" length="${elbow_width}"/>
         </geometry>
       </collision>
-      <xacro:cylinder_inertia m="1" r="${elbow_radius}" h="${elbow_width}"/>
+      <xacro:cylinder_inertia m="1.0" r="${elbow_radius}" h="${elbow_width}"/>
     </link>
+    <gazebo reference="${prefix}_elbow_link">
+      <mu>50</mu>
+      <mu2>25</mu2>
+      <kp value="50000.0"/>
+      <kd value="0.05"/>
+      <dampingFactor value="0.0"/>
+    </gazebo>
     <joint name="${prefix}_elbow_joint" type="revolute">
       <parent link="${prefix}_leg_link"/>
@@ -375,6 +208,6 @@
       <origin xyz="${-leg_length/2} 0 0" rpy="0 0 ${pi/2}"/>
       <axis xyz="1 0 0"/>
-      <limit effort="1000" lower="${-pi/2}" upper="${pi/2}" velocity="9.52"/>
-      <dynamics damping="0.0" friction="1.0"/>
+      <limit effort="1000" lower="${-pi/2}" upper="${pi/2}" velocity="0.0"/>
+      <dynamics damping="0" friction="1"/>
     </joint>
   </xacro:macro>
@@ -393,9 +226,16 @@
       <collision>
         <geometry>
-          <box size="0 0 0"/>
+          <box size="${wrist_length} ${wrist_width} ${wrist_height}"/>
         </geometry>
       </collision>
-      <xacro:box_inertia m="1" w="${wrist_width}" d="${wrist_length}" h="${wrist_height}"/>
+      <xacro:box_inertia m="1.0" w="${wrist_width}" d="${wrist_length}" h="${wrist_height}"/>
     </link>
+    <gazebo reference="${prefix}_wrist_link">
+      <mu>50</mu>
+      <mu2>25</mu2>
+      <kp value="50000.0"/>
+      <kd value="0.05"/>
+      <dampingFactor value="0.0"/>
+    </gazebo>
     <joint name="${prefix}_wrist_joint" type="fixed">
       <parent link="${prefix}_elbow_link"/>
@@ -408,5 +248,5 @@
         <origin xyz="0 0 0" rpy="0 0 0"/>
         <geometry>
-            <cylinder radius="${foot_radius}" length="${foot_width+0.001}"/>
+            <cylinder radius="${foot_radius}" length="${foot_width}"/>
         </geometry>
         <material name="black">
@@ -419,11 +259,12 @@
         </geometry>
       </collision>
-      <xacro:cylinder_inertia m="1" r="${foot_radius}" h="${foot_width}"/>
+      <xacro:cylinder_inertia m="1.0" r="${foot_radius}" h="${foot_width}"/>
     </link>
     <gazebo reference="${prefix}_foot_link">
-      <mu>100</mu>
-      <mu2>50</mu2>
-      <kp  value="1000000.0" />
-      <kd  value="1.0" />
+      <mu>50</mu>
+      <mu2>25</mu2>
+      <kp value="50000.0"/>
+      <kd value="0.05"/>
+      <dampingFactor value="0.0"/>
     </gazebo>
     <joint name="${prefix}_foot_joint" type="fixed">
