Commit message: standing?!?!?!?!?!?!

File: src/sparke_description/src/sparke_spot.urdf.xacro (robot description, xacro)
@@ -94,5 +94,5 @@
       <origin xyz="${(x_pos) * x_reflect} ${(y_pos) * y_reflect} ${z_pos-0.005}" rpy="0 0 0"/>
       <axis xyz="1 0 0"/>
-      <limit effort="1000" lower="-3.141592653589793" upper="3.141592653589793" velocity="1.5"/>
+      <limit effort="1000000" lower="-3.141592653589793" upper="3.141592653589793" velocity="1.5"/>
     </joint>
     <!-- <transmission name="${prefix}_hip_trans">
@@ -131,5 +131,5 @@
       <origin xyz="0 ${(shoulder_width/2) * y_reflect} 0" rpy="0 0 0"/>
       <axis xyz="0 1 0"/>
-      <limit effort="1000" lower="-3.141592653589793" upper="3.141592653589793" velocity="1.5"/>
+      <limit effort="1000000" lower="-3.141592653589793" upper="3.141592653589793" velocity="1.5"/>
     </joint>
     <!-- <transmission name="${prefix}_shoulder_trans">
@@ -200,5 +200,5 @@
       <origin xyz="${-leg_length/2} 0 0" rpy="0 0 ${pi/2}"/>
       <axis xyz="1 0 0"/>
-      <limit effort="1000" lower="-3.141592653589793" upper="3.141592653589793" velocity="1.5"/>
+      <limit effort="1000000" lower="-3.141592653589793" upper="3.141592653589793" velocity="1.5"/>
     </joint>
     <!-- <transmission name="${prefix}_ankle_trans">
@@ -267,5 +267,5 @@
       <axis xyz="0 1 0"/>
     </joint>
-    <gazebo reference="${prefix}_foot_link">
+    <!-- <gazebo reference="${prefix}_foot_link">
       <kp>10000000000.0</kp>
       <kd>100.0</kd>
@@ -274,5 +274,5 @@
       <minDepth>0.05</minDepth>
       <material>Gazebo/FlatBlack</material>
-    </gazebo>
+    </gazebo> -->
     <!-- <gazebo reference="${prefix}_foot_joint">
       <mu>50</mu>

Commit message: fixed origin placement in urdf

File: src/sparke_description/src/sparke_spot.urdf.xacro (robot description, xacro)
@@ -184,6 +184,6 @@
       </visual>
       <collision>
-        <geometry>
-          <origin xyz="0 0 0" rpy="0 ${pi/2} 0"/>
+        <origin xyz="0 0 0" rpy="0 ${pi/2} 0"/>
+        <geometry>
           <cylinder radius="${ankle_radius}" length="${ankle_width}"/>
         </geometry>
